File: ne5044_emulator.sch (EAGLE design)
At the start: 13 parts, among them IC2 STM8S003F3, U1 NE5044_MINIMAL_PADS, U2 SPX1117M3-L-5-0

Commit message: - Add output transistor
Parts:
- added Q1: BC847ALT1SMD, transistor-npn:BC847ALT1SMD
- added R2: 1K, rcl:R-EU_R0603
Connections:
- new net ENCODED_SIGNAL_OC: Q1.C, U1.SER_OUT
- new net N$2: Q1.B, R2.1
- net ENCODED_SIGNAL: now also R2.2; no longer U1.SER_OUT
- net GND: now also Q1.E
